File: audio_adc.kicad_sch (KiCad schematic)
At the start: 29 parts, among them J202 KLP42X-61-WW_RR, U203 PCM1802DBR, U204 PCM1802DBR

Commit message: Replace BNC connector
Replace BNC connector and change PCB size to "original" MISRC
Other:
- title: MISRC -> MISRC-PCM
Changed lines of the file:
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@@
 	(paper "A4")
 	(title_block
-		(title "MISRC")
-		(date "2024-05-10")
-		(rev "2.0")
+		(title "MISRC-PCM")
+		(date "2024-05-23")
+		(rev "2.1")
 		(comment 1 "Analog audio input + ADC")
 	)
@@
 		)
 		(instances
-			(project "MISRC_v2"
+			(project "MISRC_v2.1"
 				(path "/bc796fa4-76ff-4554-a44c-2597c6c5788e/07b85357-1780-4b3f-b9f1-20d375c30c9c"
 					(reference "#PWR0269")
@@
 		)
 		(instances
-			(project "MISRC_v2"
+			(project "MISRC_v2.1"
 				(path "/bc796fa4-76ff-4554-a44c-2597c6c5788e/07b85357-1780-4b3f-b9f1-20d375c30c9c"
 					(reference "R233")
@@
 		)
 		(instances
-			(project "MISRC_v2"
+			(project "MISRC_v2.1"
 				(path "/bc796fa4-76ff-4554-a44c-2597c6c5788e/07b85357-1780-4b3f-b9f1-20d375c30c9c"
 					(reference "#PWR0259")
@@
 		)
 		(instances
-			(project "MISRC_v2"
+			(project "MISRC_v2.1"
 				(path "/bc796fa4-76ff-4554-a44c-2597c6c5788e/07b85357-1780-4b3f-b9f1-20d375c30c9c"
 					(reference "#PWR0264")
@@
 		)
 		(instances
-			(project "MISRC_v2"
+			(project "MISRC_v2.1"
 				(path "/bc796fa4-76ff-4554-a44c-2597c6c5788e/07b85357-1780-4b3f-b9f1-20d375c30c9c"
 					(reference "R239")
@@
 		)
 		(instances
-			(project "MISRC_v2"
+			(project "MISRC_v2.1"
 				(path "/bc796fa4-76ff-4554-a44c-2597c6c5788e/07b85357-1780-4b3f-b9f1-20d375c30c9c"
 					(reference "#PWR0258")
@@
 		)
 		(instances
-			(project "MISRC_v2"
+			(project "MISRC_v2.1"
 				(path "/bc796fa4-76ff-4554-a44c-2597c6c5788e/07b85357-1780-4b3f-b9f1-20d375c30c9c"
 					(reference "C236")
@@
 		)
 		(instances
-			(project "MISRC_v2"
+			(project "MISRC_v2.1"
 				(path "/bc796fa4-76ff-4554-a44c-2597c6c5788e/07b85357-1780-4b3f-b9f1-20d375c30c9c"
 					(reference "#PWR0273")
@@
 		)
 		(instances
-			(project "MISRC_v2"
+			(project "MISRC_v2.1"
 				(path "/bc796fa4-76ff-4554-a44c-2597c6c5788e/07b85357-1780-4b3f-b9f1-20d375c30c9c"
 					(reference "R234")
@@
 		)
 		(instances
-			(project "MISRC_v2"
+			(project "MISRC_v2.1"
 				(path "/bc796fa4-76ff-4554-a44c-2597c6c5788e/07b85357-1780-4b3f-b9f1-20d375c30c9c"
 					(reference "J202")
@@
 		)
 		(instances
-			(project "MISRC_v2"
+			(project "MISRC_v2.1"
 				(path "/bc796fa4-76ff-4554-a44c-2597c6c5788e/07b85357-1780-4b3f-b9f1-20d375c30c9c"
 					(reference "C232")
@@
 		)
 		(instances
-			(project "MISRC_v2"
+			(project "MISRC_v2.1"
 				(path "/bc796fa4-76ff-4554-a44c-2597c6c5788e/07b85357-1780-4b3f-b9f1-20d375c30c9c"
 					(reference "C231")
@@
 		)
 		(instances
-			(project "MISRC_v2"
+			(project "MISRC_v2.1"
 				(path "/bc796fa4-76ff-4554-a44c-2597c6c5788e/07b85357-1780-4b3f-b9f1-20d375c30c9c"
 					(reference "C230")
@@
 		)
 		(instances
-			(project "MISRC_v2"
+			(project "MISRC_v2.1"
 				(path "/bc796fa4-76ff-4554-a44c-2597c6c5788e/07b85357-1780-4b3f-b9f1-20d375c30c9c"
 					(reference "#PWR0261")
@@
 		)
 		(instances
-			(project "MISRC_v2"
+			(project "MISRC_v2.1"
 				(path "/bc796fa4-76ff-4554-a44c-2597c6c5788e/07b85357-1780-4b3f-b9f1-20d375c30c9c"
 					(reference "#PWR0272")
@@
 		)
 		(instances
-			(project "MISRC_v2"
+			(project "MISRC_v2.1"
 				(path "/bc796fa4-76ff-4554-a44c-2597c6c5788e/07b85357-1780-4b3f-b9f1-20d375c30c9c"
 					(reference "R236")
@@
 		)
 		(instances
-			(project "MISRC_v2"
+			(project "MISRC_v2.1"
 				(path "/bc796fa4-76ff-4554-a44c-2597c6c5788e/07b85357-1780-4b3f-b9f1-20d375c30c9c"
 					(reference "U203")
@@
 		)
 		(instances
-			(project "MISRC_v2"
+			(project "MISRC_v2.1"
 				(path "/bc796fa4-76ff-4554-a44c-2597c6c5788e/07b85357-1780-4b3f-b9f1-20d375c30c9c"
 					(reference "#PWR0255")
@@
 		)
 		(instances
-			(project "MISRC_v2"
+			(project "MISRC_v2.1"
 				(path "/bc796fa4-76ff-4554-a44c-2597c6c5788e/07b85357-1780-4b3f-b9f1-20d375c30c9c"
 					(reference "#PWR0263")
@@
 		)
 		(instances
-			(project "MISRC_v2"
+			(project "MISRC_v2.1"
 				(path "/bc796fa4-76ff-4554-a44c-2597c6c5788e/07b85357-1780-4b3f-b9f1-20d375c30c9c"
 					(reference "C234")
@@
 		)
 		(instances
-			(project "MISRC_v2"
+			(project "MISRC_v2.1"
 				(path "/bc796fa4-76ff-4554-a44c-2597c6c5788e/07b85357-1780-4b3f-b9f1-20d375c30c9c"
 					(reference "#PWR0275")
@@
 		)
 		(instances
-			(project "MISRC_v2"
+			(project "MISRC_v2.1"
 				(path "/bc796fa4-76ff-4554-a44c-2597c6c5788e/07b85357-1780-4b3f-b9f1-20d375c30c9c"
 					(reference "#PWR0277")
@@
 		)
 		(instances
-			(project "MISRC_v2"
+			(project "MISRC_v2.1"
 				(path "/bc796fa4-76ff-4554-a44c-2597c6c5788e/07b85357-1780-4b3f-b9f1-20d375c30c9c"
 					(reference "C233")
@@
 		)
 		(instances
-			(project "MISRC_v2"
+			(project "MISRC_v2.1"
 				(path "/bc796fa4-76ff-4554-a44c-2597c6c5788e/07b85357-1780-4b3f-b9f1-20d375c30c9c"
 					(reference "C238")
@@
 		)
 		(instances
-			(project "MISRC_v2"
+			(project "MISRC_v2.1"
 				(path "/bc796fa4-76ff-4554-a44c-2597c6c5788e/07b85357-1780-4b3f-b9f1-20d375c30c9c"
 					(reference "C237")
@@
 		)
 		(instances
-			(project "MISRC_v2"
+			(project "MISRC_v2.1"
 				(path "/bc796fa4-76ff-4554-a44c-2597c6c5788e/07b85357-1780-4b3f-b9f1-20d375c30c9c"
 					(reference "C239")
@@
 		)
 		(instances
-			(project "MISRC_v2"
+			(project "MISRC_v2.1"
 				(path "/bc796fa4-76ff-4554-a44c-2597c6c5788e/07b85357-1780-4b3f-b9f1-20d375c30c9c"
 					(reference "#PWR0268")
@@
 		)
 		(instances
-			(project "MISRC_v2"
+			(project "MISRC_v2.1"
 				(path "/bc796fa4-76ff-4554-a44c-2597c6c5788e/07b85357-1780-4b3f-b9f1-20d375c30c9c"
 					(reference "#PWR0270")
@@
 		)
 		(instances
-			(project "MISRC_v2"
+			(project "MISRC_v2.1"
 				(path "/bc796fa4-76ff-4554-a44c-2597c6c5788e/07b85357-1780-4b3f-b9f1-20d375c30c9c"
 					(reference "#PWR0271")
@@
 		)
 		(instances
-			(project "MISRC_v2"
+			(project "MISRC_v2.1"
 				(path "/bc796fa4-76ff-4554-a44c-2597c6c5788e/07b85357-1780-4b3f-b9f1-20d375c30c9c"
 					(reference "R232")
@@
 		)
 		(instances
-			(project "MISRC_v2"
+			(project "MISRC_v2.1"
 				(path "/bc796fa4-76ff-4554-a44c-2597c6c5788e/07b85357-1780-4b3f-b9f1-20d375c30c9c"
 					(reference "R227")
@@
 		)
 		(instances
-			(project "MISRC_v2"
+			(project "MISRC_v2.1"
 				(path "/bc796fa4-76ff-4554-a44c-2597c6c5788e/07b85357-1780-4b3f-b9f1-20d375c30c9c"
 					(reference "#PWR0274")
@@
 		)
 		(instances
-			(project "MISRC_v2"
+			(project "MISRC_v2.1"
 				(path "/bc796fa4-76ff-4554-a44c-2597c6c5788e/07b85357-1780-4b3f-b9f1-20d375c30c9c"
 					(reference "R240")
@@
 		)
 		(instances
-			(project "MISRC_v2"
+			(project "MISRC_v2.1"
 				(path "/bc796fa4-76ff-4554-a44c-2597c6c5788e/07b85357-1780-4b3f-b9f1-20d375c30c9c"
 					(reference "#PWR0278")
@@
 		)
 		(instances
-			(project "MISRC_v2"
+			(project "MISRC_v2.1"
 				(path "/bc796fa4-76ff-4554-a44c-2597c6c5788e/07b85357-1780-4b3f-b9f1-20d375c30c9c"
 					(reference "C240")
@@
 		)
 		(instances
-			(project "MISRC_v2"
+			(project "MISRC_v2.1"
 				(path "/bc796fa4-76ff-4554-a44c-2597c6c5788e/07b85357-1780-4b3f-b9f1-20d375c30c9c"
 					(reference "#PWR0260")
@@
 		)
 		(instances
-			(project "MISRC_v2"
+			(project "MISRC_v2.1"
 				(path "/bc796fa4-76ff-4554-a44c-2597c6c5788e/07b85357-1780-4b3f-b9f1-20d375c30c9c"
 					(reference "#PWR0256")
@@
 		)
 		(instances
-			(project "MISRC_v2"
+			(project "MISRC_v2.1"
 				(path "/bc796fa4-76ff-4554-a44c-2597c6c5788e/07b85357-1780-4b3f-b9f1-20d375c30c9c"
 					(reference "R238")
@@
 		)
 		(instances
-			(project "MISRC_v2"
+			(project "MISRC_v2.1"
 				(path "/bc796fa4-76ff-4554-a44c-2597c6c5788e/07b85357-1780-4b3f-b9f1-20d375c30c9c"
 					(reference "#PWR0276")
@@
 		)
 		(instances
-			(project "MISRC_v2"
+			(project "MISRC_v2.1"
 				(path "/bc796fa4-76ff-4554-a44c-2597c6c5788e/07b85357-1780-4b3f-b9f1-20d375c30c9c"
 					(reference "R235")
@@
 		)
 		(instances
-			(project "MISRC_v2"
+			(project "MISRC_v2.1"
 				(path "/bc796fa4-76ff-4554-a44c-2597c6c5788e/07b85357-1780-4b3f-b9f1-20d375c30c9c"
 					(reference "R230")
@@
 		)
 		(instances
-			(project "MISRC_v2"
+			(project "MISRC_v2.1"
 				(path "/bc796fa4-76ff-4554-a44c-2597c6c5788e/07b85357-1780-4b3f-b9f1-20d375c30c9c"
 					(reference "R237")
@@
 		)
 		(instances
-			(project "MISRC_v2"
+			(project "MISRC_v2.1"
 				(path "/bc796fa4-76ff-4554-a44c-2597c6c5788e/07b85357-1780-4b3f-b9f1-20d375c30c9c"
 					(reference "#PWR0265")
@@
 		)
 		(instances
-			(project "MISRC_v2"
+			(project "MISRC_v2.1"
 				(path "/bc796fa4-76ff-4554-a44c-2597c6c5788e/07b85357-1780-4b3f-b9f1-20d375c30c9c"
 					(reference "U204")
@@
 		)
 		(instances
-			(project "MISRC_v2"
+			(project "MISRC_v2.1"
 				(path "/bc796fa4-76ff-4554-a44c-2597c6c5788e/07b85357-1780-4b3f-b9f1-20d375c30c9c"
 					(reference "#PWR0262")
@@
 		)
 		(instances
-			(project "MISRC_v2"
+			(project "MISRC_v2.1"
 				(path "/bc796fa4-76ff-4554-a44c-2597c6c5788e/07b85357-1780-4b3f-b9f1-20d375c30c9c"
 					(reference "R243")
@@
 		)
 		(instances
-			(project "MISRC_v2"
+			(project "MISRC_v2.1"
 				(path "/bc796fa4-76ff-4554-a44c-2597c6c5788e/07b85357-1780-4b3f-b9f1-20d375c30c9c"
 					(reference "#PWR0266")
@@
 		)
 		(instances
-			(project "MISRC_v2"
+			(project "MISRC_v2.1"
 				(path "/bc796fa4-76ff-4554-a44c-2597c6c5788e/07b85357-1780-4b3f-b9f1-20d375c30c9c"
 					(reference "R241")
@@
 		)
 		(instances
-			(project "MISRC_v2"
+			(project "MISRC_v2.1"
 				(path "/bc796fa4-76ff-4554-a44c-2597c6c5788e/07b85357-1780-4b3f-b9f1-20d375c30c9c"
 					(reference "C235")
@@
 		)
 		(instances
-			(project "MISRC_v2"
+			(project "MISRC_v2.1"
 				(path "/bc796fa4-76ff-4554-a44c-2597c6c5788e/07b85357-1780-4b3f-b9f1-20d375c30c9c"
 					(reference "R229")
@@
 		)
 		(instances
-			(project "MISRC_v2"
+			(project "MISRC_v2.1"
 				(path "/bc796fa4-76ff-4554-a44c-2597c6c5788e/07b85357-1780-4b3f-b9f1-20d375c30c9c"
 					(reference "#PWR0257")
@@
 		)
 		(instances
-			(project "MISRC_v2"
+			(project "MISRC_v2.1"
 				(path "/bc796fa4-76ff-4554-a44c-2597c6c5788e/07b85357-1780-4b3f-b9f1-20d375c30c9c"
 					(reference "C229")
