File: input_adc.kicad_sch (KiCad schematic)
At the start: 67 parts, among them J101 BNC_Rosenberger, J101/2 Conn_01x01_Shielded, Q101 CMPT5179, Q102 CMPT5179, SW101 SW_DIP_x04, SW102 SW_DIP_x03, SW103 SW_DIP_x03, SW104 SW_DIP_x03, SW105 SW_DIP_x02, U101 AD8138ARZ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

Commit message: Replace BNC connector
Replace BNC connector and change PCB size to "original" MISRC
Parts:
- J101: footprint Footprints:BNC Socket_mod -> Footprints:BNC_Right_Angle-DOSIN-801-0050_5pin; Manufacturer_Part_Number 5415025-2 -> DOSIN-801-0050
Other:
- title: MISRC -> MISRC-PCM
