File: power_supply.kicad_sch (KiCad schematic)
At the start: 34 parts, among them Q1 FZT690B, Q2 FZT790A, U6 TPS60401, U7 ADP7156ARDZ

Commit message: Replace BNC connector
Replace BNC connector and change PCB size to "original" MISRC
Other:
- title: MISRC -> MISRC-PCM
