File: MISRC_v2.1.kicad_pcb (KiCad board)
At the start: 2 copper layers, 146.2 x 72.6 mm, 226 parts, among them J1 Conn_01x01_Shielded, J101 BNC_Rosenberger, J101/2 Conn_01x01_Shielded, J2 Conn_01x08_Socket, J201 BNC_Rosenberger, J201/2 Conn_01x01_Shielded, J202 KLP42X-61-WW_RR, J3 GPIFII_J6, J4 GPIFII_J7, Q1 FZT690B, Q101 CMPT5179, Q102 CMPT5179, Q2 FZT790A, Q201 CMPT5179, Q202 CMPT5179, SW1 SW_Push, SW101 SW_DIP_x04, SW102 SW_DIP_x03, SW103 SW_DIP_x03, SW104 SW_DIP_x03, SW105 SW_DIP_x02, SW2 SW_DIP_x01, SW201 SW_DIP_x04, SW202 SW_DIP_x03, SW203 SW_DIP_x03, SW204 SW_DIP_x03, SW205 SW_DIP_x02, U1 4043, U101 AD8138ARZ, U102 AD9235, U2 74VHC541, U201 AD8138ARZ, U202 AD9235, U203 PCM1802DBR, U204 PCM1802DBR, U3 74VHC541, U4 74VHC541, U5 74VHC541, U6 TPS60401, U7 ADP7156ARDZ, X1 40M

Commit message: Update silkscreen
Update bottom side silkscreen
Parts:
- J202: footprint Footprints:KLP42X61WWRR -> PEPPI_FOOTPRINTS:KLP42X61WWRR
Other:
- board text added: "MISRC v2.1"
- board text removed: "MISRC v2.0"
Changed lines of the file:
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@@
 		)
 	)
-	(footprint "Footprints:KLP42X61WWRR"
+	(footprint "PEPPI_FOOTPRINTS:KLP42X61WWRR"
 		(layer "F.Cu")
 		(at 67.65 90.55 -90)
@@
 			)
 		)
-		(property "Manufacturer_Part_Number" "5415025-2"
+		(property "Manufacturer_Part_Number" "DOSIN-801-0050"
 			(at 0 0 0)
 			(unlocked yes)
@@
 			)
 		)
-		(property "Manufacturer_Part_Number" "5415025-2"
+		(property "Manufacturer_Part_Number" "DOSIN-801-0050"
 			(at 0 0 0)
 			(unlocked yes)
@@
 		)
 	)
-	(gr_text "MISRC v2.0"
+	(gr_text "MISRC v2.1"
 		(at 186.4 124.5 0)
 		(layer "B.SilkS")
